File: PCB/SimplePageTurner.kicad_sch (KiCad schematic)
At the start: 7 parts, among them SW1 SW_SPDT, SW2 SW_Push, SW3 SW_Push, SW4 SW_Push, U1 XIAO-ESP32-S3-SMD

Commit message: Added firmware
Other:
- note added: "SW 2 and 3 are page turners, SW 4 is multi fuction button."
Changed lines of the file:
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@@
 	(generator_version "10.0")
 	(paper "A4")
+	(text "SW 2 and 3 are page turners, SW 4 is multi fuction button."
+		(exclude_from_sim no)
+		(at 94.742 67.31 0)
+		(effects
+			(font
+				(size 1.27 1.27)
+			)
+		)
+	)
 	(text_box "Battery"
 		(exclude_from_sim no)
